File: startinglayout.sch (EAGLE design)
At the start: 5 parts

Commit message: I think that I'm almost done with the schematic
It needs the Li-Ion for the Matrix/Rasp/ATMega
Parts:
- removed MATRIX_FPGA: 6SLX4CPG196, xilinx_devices_V6:6SLX4CPG196
- removed RASP_PI_CAMERA: RASPI_CAM, raspberrypi_cm:RASPI_CAM
- removed RASP_PI_COMPUTING_MODULE: COMPUTE_MODULE, raspberrypi_cm:COMPUTE_MODULE
- removed RASP_PI_DISPLAY: RASPI_DSI, raspberrypi_cm:RASPI_DSI
- added C1: 470p, rcl:C-EUC0805K
- added C10, C11, C18, C2, C3, C4, C9: 100n, rcl:C-EUC0805K
- added C15: .33u, capacitor-wima:C2,5-3
- added C16, C17: 30p, rcl:C-EUC0805K
- added C19, C6, C7, C8: 4.7u, rcl:C-EUC0805K
- added C20: .1u, capacitor-wima:C2,5-3
- added C5: 1u, rcl:C-EUC0805K
- added D1, D4: B340A, SparkFun-DiscreteSemi:DIODE-SCHOTTKY_
- added D2, D3, D5, D6, D7: GREEN, led:LEDCHIP-LED0805
- added H1, H2, H3, H4: STAND-OFF, SparkFun-Hardware:STAND-OFF
- added J1: 3x2 M, SmartPrj:PINHD-2X3
- added J2: S2B-PH-SM4-TB(LF)(SN), SparkFun-Connectors:M02-JST-2MM-SMT
- added J3: 629105136821, Wurth_Elektronik_Electromechanic_Input-Output_Connectors_rev19b:629105136821
- added Q1, Q10, Q2, Q7: 2N706, transistor-npn:2N706
- added Q11, Q3, Q4, Q8: BUZ23, transistor-fet:BUZ23
- added Q12, Q5, Q6, Q9: BUZ171, transistor-fet:BUZ171
- added R1, R10, R11, R12, R8: 1K, rcl:R-US_R0805
- added R13, R14, R16, R17, R18, R19, R21, R22: 10k, rcl:R-US_0204/5
- added R15, R20, R7, R9: 2.2k, rcl:R-US_0204/5
- added R2, R3, R6: 10K, rcl:R-US_R0805
- added R4, R5: 22, rcl:R-US_R0805
- added SV1: ATMEGA_DRIVER_CONNECTOR, con-lstb:MA04-1
- added SW1: AYZ0202AGRLC, SparkFun-Electromechanical:SWITCH-DPDTSMD
- added SW2: !RESET, SparkFun-Electromechanical:SWITCH-MOMENTARY-2SMD
- added TP3: TPPAD1-13, testpad:TPPAD1-13
- added TX_RASP: RASP_TO_ATMEG_CONNECTOR, con-garry:332-04
- added U1: MCP73831, SparkFun-PowerIC:MCP73831
- added U2: MIC5219, SparkFun-PowerIC:V_REG_MIC5219SMD
- added U3: ATMEGA32U4-AUR, SparkFun-IC-Microcontroller:ATMEGA32U4TQFP-44
- added VOLTAGE_REGULATOR: 7805ABV, linear:7805H
- added X2: 16 MHz, SparkFun-Clocks:CRYSTALSMD-HC49UP
Connections:
- new net !RESET: J1.5, R3.1, SW2.2, TP3.TP, U3.!RESET
- new net +5V: C15.1, VOLTAGE_REGULATOR.VI
- new net AREF: C4.1, U3.AREF
- new net CONTROL_L_BACKWARD: Q8.G, R16.1, R7.1
- new net CONTROL_L_FORWARD: Q3.G, R13.1, R15.1
- new net CONTROL_R_BACKWARD: Q11.G, R21.1, R9.1
- new net CONTROL_R_FORWARD: Q4.G, R18.1, R20.1
- new net D+: R5.2, U3.D+
- new net D-: R4.2, U3.D-
- new net D13#/USER_LED: R11.2, U3.PC7
- new net D14/MISO: J1.1, U3.PB3(MISO)
- new net D15/SCK: J1.3, U3.PB1(SCK)
- new net D16/MOSI: J1.4, U3.PB2(MOSI)
- new net D17/RX-LED: D6.C, U3.PB0(SS)
- new net GND: C1.2, C10.2, C11.2, C16.2, C17.2, C18.2, C19.2, C2.2, C3.2, C4.2, C5.2, C6.2, C7.2, C8.2, C9.2, D2.C, D3.C, J1.6, J2.2, J3.GND, R2.1, R6.1, SW1.3, SW2.1, U1.VSS, U2.GND, U3.GND@15, U3.GND@23, U3.GND@35, U3.GND@43, U3.UGND
- new net GPIO_GCLK: MATRIX_TO_RASP_PI_CONNECTOR.GP4
- new net H_BRIDGE_POWER: C20.1, VOLTAGE_REGULATOR.VO
- new net H_BRIDGE_POWER(5V): Q12.S, Q5.S, Q6.S, Q9.S, R14.2, R17.2, R19.2, R22.2
- new net MATRIX_FPGA: MATRIX_TO_RASP_PI_CONNECTOR.CE0, MATRIX_TO_RASP_PI_CONNECTOR.CE1, MATRIX_TO_RASP_PI_CONNECTOR.GP18#, MATRIX_TO_RASP_PI_CONNECTOR.GP26
- new net MATRIX_JTAG_TCK: MATRIX_TO_RASP_PI_CONNECTOR.GP27
- new net MATRIX_JTAG_TDI: MATRIX_TO_RASP_PI_CONNECTOR.GP23
- new net MATRIX_JTAG_TDO: MATRIX_TO_RASP_PI_CONNECTOR.GP22
- new net MATRIX_JTAG_TMS: MATRIX_TO_RASP_PI_CONNECTOR.GP17
- new net MATRIX_SCLK_I2C: MATRIX_TO_RASP_PI_CONNECTOR.SCL
- new net MATRIX_SDA_I2C: MATRIX_TO_RASP_PI_CONNECTOR.SDA
- new net MATRIX_SPI_CLK: MATRIX_TO_RASP_PI_CONNECTOR.MOSI
- new net MATRIX_SPI_MISO: MATRIX_TO_RASP_PI_CONNECTOR.MISO
- new net MATRIX_SPI_MOSI: MATRIX_TO_RASP_PI_CONNECTOR.SCLK
- new net MCPPROG: R2.2, U1.PROG
- new net MIC-BP: C1.1, U2.BP
- new net MIC-EN: SW1.2, U2.EN
- new net N$1: Q1.C, Q5.G, R14.1
- new net N$10: MATRIX_TO_RASP_PI_CONNECTOR.GND@14, MATRIX_TO_RASP_PI_CONNECTOR.GND@20, MATRIX_TO_RASP_PI_CONNECTOR.GND@25, MATRIX_TO_RASP_PI_CONNECTOR.GND@30, MATRIX_TO_RASP_PI_CONNECTOR.GND@34, MATRIX_TO_RASP_PI_CONNECTOR.GND@39, MATRIX_TO_RASP_PI_CONNECTOR.GND@6, MATRIX_TO_RASP_PI_CONNECTOR.GND@9
- new net N$11: Q7.B, R15.2
- new net N$12: Q10.C, Q12.G, R22.1
- new net N$13: D3.A, R11.1
- new net N$14: C18.1, J3.SHIELD
- new net N$15: D6.A, R8.1
- new net N$16: D7.A, R12.1
- new net N$17: Q8.D, Q9.D
- new net N$18: Q11.D, Q12.D
- new net N$19: J3.D-, R4.1
- new net N$2: Q2.C, Q6.G, R19.1
- new net N$20: J3.D+, R5.1
- new net N$21: Q10.B, R20.2
- new net N$22: Q2.B, R9.2
- new net N$23: U3.PE6
- new net N$24: U3.PB4(ADC11)
- new net N$25: U3.PB5(ADC12)
- new net N$26: U3.PC6
- new net N$27: U3.PD4(ADC8)
- new net N$28: U3.PD0(SCL)
- new net N$29: U3.PD1(SDA)
- new net N$3: D5.A, R1.1
- new net N$30: U3.PD3(TX)
- new net N$31: U3.PD2(RX)
- new net N$32: MATRIX_TO_RASP_PI_CONNECTOR.GP5
- new net N$33: MATRIX_TO_RASP_PI_CONNECTOR.GP6
- new net N$34: MATRIX_TO_RASP_PI_CONNECTOR.GP12
- new net N$35: MATRIX_TO_RASP_PI_CONNECTOR.GP13
- new net N$36: MATRIX_TO_RASP_PI_CONNECTOR.GP16
- new net N$37: MATRIX_TO_RASP_PI_CONNECTOR.GP19
- new net N$38: MATRIX_TO_RASP_PI_CONNECTOR.GP20
- new net N$39: MATRIX_TO_RASP_PI_CONNECTOR.GP21
- new net N$4: D5.C, U1.STAT
- new net N$40: U3.PF7(ADC7)
- new net N$41: MATRIX_TO_RASP_PI_CONNECTOR.5V@2, MATRIX_TO_RASP_PI_CONNECTOR.5V@4
- new net N$42: U3.PF6(ADC6)
- new net N$43: U3.PF5(ADC5)
- new net N$44: U3.PF4(ADC4)
- new net N$45: U3.PF1(ADC1)
- new net N$46: U3.PF0(ADC0)
- new net N$5: Q1.B, R7.2
- new net N$6: Q7.C, Q9.G, R17.1
- new net N$7: D2.A, R10.1
- new net N$8: Q4.D, Q6.D
- new net N$9: Q3.D, Q5.D
- new net NC_(ESP): MATRIX_TO_RASP_PI_CONNECTOR.GP24, MATRIX_TO_RASP_PI_CONNECTOR.GP25
- new net PE2/!HWB: R6.2, U3.PE2/!HWB
- new net PWM_1: U3.PB6(ADC13)
- new net PWM_2: U3.PB7
- new net PWM_3: U3.PD6(ADC9)
- new net PWM_4: U3.PD7(ADC10)
- new net PWRIN: C7.1, D1.C, D4.C, SW1.1, U2.IN
- new net RX_RASP: MATRIX_TO_RASP_PI_CONNECTOR.RXI
- new net TX_LED: D7.C, U3.PD5
- new net TX_RASP: MATRIX_TO_RASP_PI_CONNECTOR.TXO
- new net UCAP: C5.1, U3.UCAP
- new net VBUS: C19.1, D4.A, J3.VBUS, R1.2, U1.VIN, U3.UVCC, U3.VBUS
- new net V_BATT: C6.1, D1.A, J2.1, U1.VBAT
- new net XTAL1: C17.1, U3.XTAL1, X2.2
- new net XTAL2: C16.1, U3.XTAL2, X2.1
- net 0: now also C15.2, C20.2, Q1.E, Q10.E, Q11.S, Q2.E, Q3.S, Q4.S, Q7.E, Q8.S, R13.2, R16.2, R18.2, R21.2, VOLTAGE_REGULATOR.GND; no longer MATRIX_TO_RASP_PI_CONNECTOR.GND@14, MATRIX_TO_RASP_PI_CONNECTOR.GND@20, MATRIX_TO_RASP_PI_CONNECTOR.GND@25, MATRIX_TO_RASP_PI_CONNECTOR.GND@30, MATRIX_TO_RASP_PI_CONNECTOR.GND@34, MATRIX_TO_RASP_PI_CONNECTOR.GND@39, MATRIX_TO_RASP_PI_CONNECTOR.GND@6, MATRIX_TO_RASP_PI_CONNECTOR.GND@9
- net 3.3V: now also C10.1, C11.1, C2.1, C3.1, C8.1, C9.1, J1.2, R10.2, R12.2, R3.2, R8.2, U2.OUT, U3.AVCC@24, U3.AVCC@44, U3.VCC@14, U3.VCC@34
Other:
- note added: "ATMEGA PROCESSOR IN LILYPAD SCHEMATIC"
- note added: "CHARGE"
- note added: "ICSP"
- note added: "M3 / #4-40 mounting holes"
- note added: "MATRIX VOICE SOUND SENSOR"
- note added: "MATRIX_TO_RASP_PI_CONNECTOR"
- note added: "MOTOR"
- note added: "MOTOR ACTUATORS + DRIVERS"
- note added: "Originally taken from AndrewGreenburg/Eaglecad-things repo"
- note added: "Originally taken from Arduino Lilypad Rev 10 Licensed under Creative Commons Attribution ShareAlike (CC BY-SA)"
- note added: "POWER"
- note added: "PWM_1"
- note added: "PWM_2"
- note added: "PWM_3"
- note added: "PWM_4"
- note added: "RASPBERRY PI 3 SOUND SENSOR EXTENSION"
- note added: "RASP_ATMEGA_UART_CONNECTOR"
- note added: "REQUIRED to program ATMEGA328P"
- note added: "RX_ATMEGA"
- note added: "RX_RASP"
- note added: "TX_ATMEGA"
- note added: "TX_RASP"
- note added: "USB RX"
- note added: "USB TX"
- note added: "USER"
- moved on the sheet: MATRIX_TO_RASP_PI_CONNECTOR

Commit message: Added in power supply, reduced PWM channels, added in UART (from ATmega), and converted H Bridges
Parts:
- removed Q10, Q7: 2N706, transistor-npn:2N706
- removed Q11, Q8: BUZ23, transistor-fet:BUZ23
- removed Q12, Q9: BUZ171, transistor-fet:BUZ171
- removed R16, R17, R18, R21, R22: 10k, rcl:R-US_0204/5
- removed R20: 2.2k, rcl:R-US_0204/5
- Q3, Q4: value BUZ23 -> TN0602N3; device transistor-fet:BUZ23 -> transistor-fet:TN0602N3
- R15: value 2.2k -> 10k
Connections:
- net N$30 renamed TX_ATMEGA?
- net N$31 renamed RX_ATMEGA?
- net PWM_1 renamed PWM_1?
- net PWM_2 renamed PWM_2?
- net RX_RASP renamed RX_RASP?
- net TX_RASP renamed TX_RASP?
- removed net CONTROL_L_BACKWARD: Q8.G, R16.1, R7.1
- removed net CONTROL_L_FORWARD: Q3.G, R13.1, R15.1
- removed net CONTROL_R_BACKWARD: Q11.G, R21.1, R9.1
- removed net CONTROL_R_FORWARD: Q4.G, R18.1, R20.1
- removed net N$17: Q8.D, Q9.D
- removed net N$21: Q10.B, R20.2
- new net CONTROL_L: Q4.G, R15.1, R7.1
- new net CONTROL_R: Q3.G, R13.1, R9.1
- net 0: no longer Q10.E, Q11.S, Q3.S, Q4.S, Q7.E, Q8.S, R13.2, R16.2, R18.2, R21.2
- net H_BRIDGE_POWER(5V): no longer Q12.S, Q9.S, R17.2, R22.2
- net N$11: now also Q4.S; no longer Q7.B
- net N$12: now also Q3.D; no longer Q10.C, Q12.G, R22.1
- net N$18: now also Q3.S, R13.2; no longer Q11.D, Q12.D
- net N$6: now also Q4.D; no longer Q7.C, Q9.G, R17.1
- net N$8: no longer Q4.D
- net N$9: no longer Q3.D
Other:
- note added: "(7.6V Li-Ion battery pack)"
- note added: "*The Rasp Pi connector on the Matrix Voice has unused UART pins on it that we're hoping to utilize for the Rasp Pi and ATmega32U connection"
- note added: "I hope that these are the right pins for doing UART between the Rasp PI and the ATmega as well as the right PWM capable pins. Are there other UART or PWM pins that we need to be aware of?"
- note added: "Li-Ion source for Matrix Voice, Rasp. Pi, and ATMega setup"
- note added: "POWER IN"
- note added: "The two motors shown are for the left and right tires of the chassis Using half H-bridges (only want to turn in forward direction) and PWM we're hoping that we'll be able to control said motors."
- note removed: "PWM_3"
- note removed: "PWM_4"
- moved on the sheet: R13, R15

Commit message: Added in the H Bridge ICs and removed what was before
Parts:
- removed Q1, Q2: 2N706, transistor-npn:2N706
- removed Q3, Q4: TN0602N3, transistor-fet:TN0602N3
- removed Q5, Q6: BUZ171, transistor-fet:BUZ171
- removed R13, R14, R15, R19: 10k, rcl:R-US_0204/5
- removed R7, R9: 2.2k, rcl:R-US_0204/5
- added LEFT_HBRIDGE_DRIVER, RIGHT_HBRIDGE_DRIVER: BD6230F, rohm:BD6230F
Connections:
- removed net CONTROL_L: Q4.G, R15.1, R7.1
- removed net CONTROL_R: Q3.G, R13.1, R9.1
- removed net H_BRIDGE_POWER(5V): Q5.S, Q6.S, R14.2, R19.2
- removed net N$1: Q1.C, Q5.G, R14.1
- removed net N$11: Q4.S, R15.2
- removed net N$12: Q3.D
- removed net N$18: Q3.S, R13.2
- removed net N$2: Q2.C, Q6.G, R19.1
- removed net N$22: Q2.B, R9.2
- removed net N$6: Q4.D
- removed net N$9: Q5.D
- new net LEFT_MOTOR: LEFT_HBRIDGE_DRIVER.OUT1, LEFT_HBRIDGE_DRIVER.OUT2
- new net PWM_1: LEFT_HBRIDGE_DRIVER.FIN
- new net PWM_2: LEFT_HBRIDGE_DRIVER.RIN
- new net RIGHT_MOTOR: RIGHT_HBRIDGE_DRIVER.OUT1, RIGHT_HBRIDGE_DRIVER.OUT2
- net 0: now also LEFT_HBRIDGE_DRIVER.GND, RIGHT_HBRIDGE_DRIVER.GND; no longer Q1.E, Q2.E
- net N$5: now also LEFT_HBRIDGE_DRIVER.VCC@1, LEFT_HBRIDGE_DRIVER.VCC@2; no longer Q1.B, R7.2
- net N$8: now also RIGHT_HBRIDGE_DRIVER.VCC@1, RIGHT_HBRIDGE_DRIVER.VCC@2; no longer Q6.D
- net PWM_3: now also RIGHT_HBRIDGE_DRIVER.FIN
- net PWM_4: now also RIGHT_HBRIDGE_DRIVER.RIN
Other:
- note added: "(7.4V Li-Ion Battery pack)"
- note added: "5V"
- note added: "PWM_3"
- note added: "PWM_4"
- note removed: "(7.6V Li-Ion battery pack)"
- note removed: "MOTOR"
