File: forpcblayout.sch (EAGLE design)
At the start: 51 parts, among them J1 3x2 M, J2 S2B-PH-SM4-TB(LF)(SN), J3 629105136821, SW1 AYZ0202AGRLC, SW2 !RESET, U1 MCP73831, U2 MIC5219, U3 ATMEGA32U4-AUR, X2 16 MHz

Commit message: Inluded H-bridge ICs, more connectors, and replaced UART with I2C
Parts:
- removed SV1: ATMEGA_DRIVER_CONNECTOR, con-lstb:MA04-1
- removed TX_RASP: RASP_TO_ATMEG_CONNECTOR, con-garry:332-04
- added LEFT_HBRIDGE_DRIVER, RIGHT_HBRIDGE_DRIVER: BD6230F, rohm:BD6230F
- added MOTOR_CONNECTOR, PWM_CONNECTOR: (no value), con-lstb:MA04-2
- added R7, R9: 1K, rcl:R-US_R0805
- added RASP_TO_ATMEGA_I2C_CONNECTOR: (no value), con-lstb:MA04-1
Connections:
- removed net N$28: U3.PD0(SCL)
- removed net N$29: U3.PD1(SDA)
- removed net PWM_1?: SV1.1, U3.PB6(ADC13)
- removed net PWM_2?: SV1.2, U3.PB7
- removed net RX_ATMEGA?: TX_RASP-4.S, U3.PD2(RX)
- removed net TX_ATMEGA?: TX_RASP-2.S, U3.PD3(TX)
- new net LEFT_MOTOR1: LEFT_HBRIDGE_DRIVER.OUT1, MOTOR_CONNECTOR.7, MOTOR_CONNECTOR.8
- new net LEFT_MOTOR2: LEFT_HBRIDGE_DRIVER.OUT2, MOTOR_CONNECTOR.5, MOTOR_CONNECTOR.6
- new net NC: U3.PD2(RX), U3.PD3(TX)
- new net PWM_1: LEFT_HBRIDGE_DRIVER.FIN, PWM_CONNECTOR.7, PWM_CONNECTOR.8, U3.PB6(ADC13)
- new net PWM_2: LEFT_HBRIDGE_DRIVER.RIN, PWM_CONNECTOR.5, PWM_CONNECTOR.6, U3.PB7
- new net RIGHT_MOTOR1: MOTOR_CONNECTOR.3, MOTOR_CONNECTOR.4, RIGHT_HBRIDGE_DRIVER.OUT1
- new net RIGHT_MOTOR2: MOTOR_CONNECTOR.1, MOTOR_CONNECTOR.2, RIGHT_HBRIDGE_DRIVER.OUT2
- new net SCL: R7.1, RASP_TO_ATMEGA_I2C_CONNECTOR.1, RASP_TO_ATMEGA_I2C_CONNECTOR.2, U3.PD0(SCL)
- new net SDA: R9.1, RASP_TO_ATMEGA_I2C_CONNECTOR.3, RASP_TO_ATMEGA_I2C_CONNECTOR.4, U3.PD1(SDA)
- net (5V@2.1A): now also R7.2, R9.2
- net 0: now also LEFT_HBRIDGE_DRIVER.GND, RIGHT_HBRIDGE_DRIVER.GND
- net H_BRIDGE_POWER: now also LEFT_HBRIDGE_DRIVER.VCC@1, LEFT_HBRIDGE_DRIVER.VCC@2, RIGHT_HBRIDGE_DRIVER.VCC@1, RIGHT_HBRIDGE_DRIVER.VCC@2
- net PWM_3: now also PWM_CONNECTOR.3, PWM_CONNECTOR.4, RIGHT_HBRIDGE_DRIVER.FIN; no longer SV1.3
- net PWM_4: now also PWM_CONNECTOR.1, PWM_CONNECTOR.2, RIGHT_HBRIDGE_DRIVER.RIN
Other:
- note added: "FROM PI"
- note added: "MOTOR ACTUATORS + DRIVERS"
- note added: "The two motors shown are for the left and right tires of the chassis Using half H-bridges (only want to turn in forward direction) and PWM we're hoping that we'll be able to control said motors."
- note added: "ZXMHC3F381N8"
- note removed: "*The Rasp Pi connector on the Matrix Voice has unused UART pins on it that we're hoping to utilize for the Rasp Pi and ATmega32U connection"
- note removed: "I hope that these are the right pins for doing UART between the Rasp PI and the ATmega as well as the right PWM capable pins. Are there other UART or PWM pins that we need to be aware of?"
- note removed: "PWM_1"
- note removed: "PWM_2"
- note removed: "PWM_3"
- note removed: "PWM_4"
- note removed: "RASP_ATMEGA_UART_CONNECTOR"
- note removed: "RX_ATMEGA"
- note removed: "RX_RASP"
- note removed: "TX_ATMEGA"
- note removed: "TX_RASP"
- moved on the sheet: C15, C20, VOLTAGE_REGULATOR

Commit message: Added in connector for Pi to ATMega as  well as battery for the schematic
Mounting holes line up (more or less) with the Pi now
We still need the right H Bridge Driver ICs, check GNDing, adding in vias for ea. GND connection, and check up on decoupling caps for power sources
Parts:
- removed RASP_TO_ATMEGA_I2C_CONNECTOR: (no value), con-lstb:MA04-1
- added MOTOR_BATTERY_CONNECTOR: (no value), con-lstb:MA04-1
- added SV1: (no value), con-lsta:FE20-2
- VOLTAGE_REGULATOR: value 7805ABV -> LM7805ABV
Connections:
- removed net +5V: C15.1, VOLTAGE_REGULATOR.VI
- removed net SCL: R7.1, RASP_TO_ATMEGA_I2C_CONNECTOR.1, RASP_TO_ATMEGA_I2C_CONNECTOR.2, U3.PD0(SCL)
- new net 7.4V_FROM_BATT: C15.1, MOTOR_BATTERY_CONNECTOR.4, VOLTAGE_REGULATOR.VI
- new net N$1: MOTOR_BATTERY_CONNECTOR.2, MOTOR_BATTERY_CONNECTOR.3
- new net N$2: PWM_CONNECTOR.7, PWM_CONNECTOR.8
- new net N$5: PWM_CONNECTOR.1, PWM_CONNECTOR.2
- new net N$6: PWM_CONNECTOR.3, PWM_CONNECTOR.4
- new net N$8: PWM_CONNECTOR.5, PWM_CONNECTOR.6
- new net POWER_IN: C10.1, C11.1, C2.1, C3.1, SV1.40, U3.AVCC@24, U3.AVCC@44, U3.VCC@14, U3.VCC@34
- new net SCLK: R7.1, SV1.35, U3.PD0(SCL)
- net (5V@2.1A): no longer C10.1, C11.1, C2.1, C3.1, U3.AVCC@24, U3.AVCC@44, U3.VCC@14, U3.VCC@34
- net 0: no longer C15.2, C20.2, VOLTAGE_REGULATOR.GND
- net GND: now also C15.2, C20.2, MOTOR_BATTERY_CONNECTOR.1, SV1.31, VOLTAGE_REGULATOR.GND
- net PWM_1: no longer PWM_CONNECTOR.7, PWM_CONNECTOR.8
- net PWM_2: no longer PWM_CONNECTOR.5, PWM_CONNECTOR.6
- net PWM_3: no longer PWM_CONNECTOR.3, PWM_CONNECTOR.4
- net PWM_4: no longer PWM_CONNECTOR.1, PWM_CONNECTOR.2
- net SDA: now also SV1.37; no longer RASP_TO_ATMEGA_I2C_CONNECTOR.3, RASP_TO_ATMEGA_I2C_CONNECTOR.4
Other:
- note added: "(5V@2.1A)"
- note added: "USB_POWER"
- note removed: "FROM PI"
- note removed: "Li-Ion source for Matrix Voice, Rasp. Pi, and ATMega setup"
- note removed: "POWER"
- note removed: "POWER IN"
- moved on the sheet: PWM_CONNECTOR
